File: kicad/switchernor.kicad_pcb (KiCad board)
At the start: 2 copper layers, 15 parts, among them J1 Conn_01x09_Pin, J2 Conn_01x09_Pin, U1 4051, U10 74HC595, U11 74HC595, U12 74HC595, U2 4051, U3 4051, U4 4051, U5 4051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

Commit message: Arduino added
Parts:
- moved J1 76.1 mm to (160.9, 50.9)
- moved J2 49.5 mm to (96.3, 51.2)
Changed lines of the file:
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@@
   )
   (footprint "Connector_PinHeader_2.54mm:PinHeader_2x05_P2.54mm_Vertical" (layer "F.Cu")
-    (at 84.841 47.63 90)
+    (at 160.914 50.932 90)
     (descr "Through hole straight pin header, 2x05, 2.54mm pitch, double rows")
     (tags "Through hole pin header THT 2x05 2.54mm double row")
@@
   )
   (footprint "Connector_PinHeader_2.54mm:PinHeader_2x05_P2.54mm_Vertical" (layer "F.Cu")
-    (at 145.542 46.101 90)
+    (at 96.266 51.181 90)
     (descr "Through hole straight pin header, 2x05, 2.54mm pitch, double rows")
     (tags "Through hole pin header THT 2x05 2.54mm double row")
